File: PCB/swiss army pcb/pi_pico.kicad_sch (KiCad schematic)
At the start: 15 parts, among them J7 Conn_01x07_Pin, J8 I2C Display, SW1 SW_SPDT, U3 Pico

Commit message: tidy up
Parts:
- J7: footprint reciever:BOB-00544 MicroSD -> things:BOB-00544 MicroSD
- J8: footprint reciever:SDD1306 -> things:SDD1306
- U3: footprint reciever:RPi_Pico_SMD_TH -> things:RPi_Pico_SMD_TH
Changed lines of the file:
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@@
         )
       )
-      (project "pico_rx"
+      (project "things"
         (path "/b6f73a49-ac1f-4895-a0f9-8f6954ee587f/ef5e145d-7cd2-41fd-85f8-55f3445b8dc3"
           (reference "H4") (unit 1)
@@
       (effects (font (size 1.27 1.27)))
     )
-    (property "Footprint" "reciever:RPi_Pico_SMD_TH" (at 142.24 77.47 0)
+    (property "Footprint" "things:RPi_Pico_SMD_TH" (at 142.24 77.47 0)
       (effects (font (size 1.27 1.27)) hide)
     )
@@
     (pin "9")
     (instances
-      (project "pico_rx"
+      (project "things"
         (path "/b6f73a49-ac1f-4895-a0f9-8f6954ee587f/ef5e145d-7cd2-41fd-85f8-55f3445b8dc3"
           (reference "U3") (unit 1)
@@
     (pin "3")
     (instances
-      (project "pico_rx"
+      (project "things"
         (path "/b6f73a49-ac1f-4895-a0f9-8f6954ee587f/ef5e145d-7cd2-41fd-85f8-55f3445b8dc3"
           (reference "SW1") (unit 1)
@@
         )
       )
-      (project "pico_rx"
+      (project "things"
         (path "/b6f73a49-ac1f-4895-a0f9-8f6954ee587f/ef5e145d-7cd2-41fd-85f8-55f3445b8dc3"
           (reference "SW2") (unit 1)
@@
         )
       )
-      (project "pico_rx"
+      (project "things"
         (path "/b6f73a49-ac1f-4895-a0f9-8f6954ee587f/ef5e145d-7cd2-41fd-85f8-55f3445b8dc3"
           (reference "J6") (unit 1)
@@
         )
       )
-      (project "pico_rx"
+      (project "things"
         (path "/b6f73a49-ac1f-4895-a0f9-8f6954ee587f/ef5e145d-7cd2-41fd-85f8-55f3445b8dc3"
           (reference "H3") (unit 1)
@@
         )
       )
-      (project "pico_rx"
+      (project "things"
         (path "/b6f73a49-ac1f-4895-a0f9-8f6954ee587f/ef5e145d-7cd2-41fd-85f8-55f3445b8dc3"
           (reference "#PWR017") (unit 1)
@@
         )
       )
-      (project "pico_rx"
+      (project "things"
         (path "/b6f73a49-ac1f-4895-a0f9-8f6954ee587f/ef5e145d-7cd2-41fd-85f8-55f3445b8dc3"
           (reference "#PWR015") (unit 1)
@@
         )
       )
-      (project "pico_rx"
+      (project "things"
         (path "/b6f73a49-ac1f-4895-a0f9-8f6954ee587f/ef5e145d-7cd2-41fd-85f8-55f3445b8dc3"
           (reference "#PWR016") (unit 1)
@@
         )
       )
-      (project "pico_rx"
+      (project "things"
         (path "/b6f73a49-ac1f-4895-a0f9-8f6954ee587f/ef5e145d-7cd2-41fd-85f8-55f3445b8dc3"
           (reference "#PWR013") (unit 1)
@@
       (effects (font (size 1.27 1.27)))
     )
-    (property "Footprint" "reciever:BOB-00544 MicroSD" (at 57.15 170.815 0)
+    (property "Footprint" "things:BOB-00544 MicroSD" (at 57.15 170.815 0)
       (effects (font (size 1.27 1.27)) hide)
     )
@@
     (pin "7")
     (instances
-      (project "pico_rx"
+      (project "things"
         (path "/b6f73a49-ac1f-4895-a0f9-8f6954ee587f/ef5e145d-7cd2-41fd-85f8-55f3445b8dc3"
           (reference "J7") (unit 1)
@@
         )
       )
-      (project "pico_rx"
+      (project "things"
         (path "/b6f73a49-ac1f-4895-a0f9-8f6954ee587f/ef5e145d-7cd2-41fd-85f8-55f3445b8dc3"
           (reference "#PWR022") (unit 1)
@@
         )
       )
-      (project "pico_rx"
+      (project "things"
         (path "/b6f73a49-ac1f-4895-a0f9-8f6954ee587f/ef5e145d-7cd2-41fd-85f8-55f3445b8dc3"
           (reference "#PWR021") (unit 1)
@@
         )
       )
-      (project "pico_rx"
+      (project "things"
         (path "/b6f73a49-ac1f-4895-a0f9-8f6954ee587f/ef5e145d-7cd2-41fd-85f8-55f3445b8dc3"
           (reference "#PWR026") (unit 1)
@@
         )
       )
-      (project "pico_rx"
+      (project "things"
         (path "/b6f73a49-ac1f-4895-a0f9-8f6954ee587f/ef5e145d-7cd2-41fd-85f8-55f3445b8dc3"
           (reference "#PWR018") (unit 1)
@@
       (effects (font (size 1.27 1.27)) (justify left))
     )
-    (property "Footprint" "reciever:SDD1306" (at 257.81 59.69 0)
+    (property "Footprint" "things:SDD1306" (at 257.81 59.69 0)
       (effects (font (size 1.27 1.27)) hide)
     )
@@
     (pin "4")
     (instances
-      (project "pico_rx"
+      (project "things"
         (path "/b6f73a49-ac1f-4895-a0f9-8f6954ee587f/ef5e145d-7cd2-41fd-85f8-55f3445b8dc3"
           (reference "J8") (unit 1)
@@
         )
       )
-      (project "pico_rx"
+      (project "things"
         (path "/b6f73a49-ac1f-4895-a0f9-8f6954ee587f/ef5e145d-7cd2-41fd-85f8-55f3445b8dc3"
           (reference "FB1") (unit 1)
@@
         )
       )
-      (project "pico_rx"
+      (project "things"
         (path "/b6f73a49-ac1f-4895-a0f9-8f6954ee587f/ef5e145d-7cd2-41fd-85f8-55f3445b8dc3"
           (reference "#PWR012") (unit 1)
@@
         )
       )
-      (project "pico_rx"
+      (project "things"
         (path "/b6f73a49-ac1f-4895-a0f9-8f6954ee587f/ef5e145d-7cd2-41fd-85f8-55f3445b8dc3"
           (reference "#PWR020") (unit 1)
@@
         )
       )
-      (project "pico_rx"
+      (project "things"
         (path "/b6f73a49-ac1f-4895-a0f9-8f6954ee587f/ef5e145d-7cd2-41fd-85f8-55f3445b8dc3"
           (reference "SW4") (unit 1)
@@
         )
       )
-      (project "pico_rx"
+      (project "things"
         (path "/b6f73a49-ac1f-4895-a0f9-8f6954ee587f/ef5e145d-7cd2-41fd-85f8-55f3445b8dc3"
           (reference "FB2") (unit 1)
@@
         )
       )
-      (project "pico_rx"
+      (project "things"
         (path "/b6f73a49-ac1f-4895-a0f9-8f6954ee587f/ef5e145d-7cd2-41fd-85f8-55f3445b8dc3"
           (reference "#PWR014") (unit 1)
@@
         )
       )
-      (project "pico_rx"
+      (project "things"
         (path "/b6f73a49-ac1f-4895-a0f9-8f6954ee587f/ef5e145d-7cd2-41fd-85f8-55f3445b8dc3"
           (reference "#PWR011") (unit 1)
@@
         )
       )
-      (project "pico_rx"
+      (project "things"
         (path "/b6f73a49-ac1f-4895-a0f9-8f6954ee587f/ef5e145d-7cd2-41fd-85f8-55f3445b8dc3"
           (reference "H1") (unit 1)
@@
         )
       )
-      (project "pico_rx"
+      (project "things"
         (path "/b6f73a49-ac1f-4895-a0f9-8f6954ee587f/ef5e145d-7cd2-41fd-85f8-55f3445b8dc3"
           (reference "#PWR023") (unit 1)
@@
         )
       )
-      (project "pico_rx"
+      (project "things"
         (path "/b6f73a49-ac1f-4895-a0f9-8f6954ee587f/ef5e145d-7cd2-41fd-85f8-55f3445b8dc3"
           (reference "SW5") (unit 1)
@@
         )
       )
-      (project "pico_rx"
+      (project "things"
         (path "/b6f73a49-ac1f-4895-a0f9-8f6954ee587f/ef5e145d-7cd2-41fd-85f8-55f3445b8dc3"
           (reference "#PWR019") (unit 1)
@@
         )
       )
-      (project "pico_rx"
+      (project "things"
         (path "/b6f73a49-ac1f-4895-a0f9-8f6954ee587f/ef5e145d-7cd2-41fd-85f8-55f3445b8dc3"
           (reference "#PWR024") (unit 1)
@@
         )
       )
-      (project "pico_rx"
+      (project "things"
         (path "/b6f73a49-ac1f-4895-a0f9-8f6954ee587f/ef5e145d-7cd2-41fd-85f8-55f3445b8dc3"
           (reference "H2") (unit 1)
@@
         )
       )
-      (project "pico_rx"
+      (project "things"
         (path "/b6f73a49-ac1f-4895-a0f9-8f6954ee587f/ef5e145d-7cd2-41fd-85f8-55f3445b8dc3"
           (reference "SW3") (unit 1)
