File: PCB/swiss army pcb/audio.kicad_sch (KiCad schematic)
At the start: 27 parts, among them U1 MCP6002-xSN, U2 TPA2012D2RTJT

Commit message: tidy up
Parts:
- J? (x2): footprint reciever:jack3.5mm switched -> things:jack3.5mm switched
- U2: footprint reciever:QFN50P400X400X80-21N270X270 -> things:QFN50P400X400X80-21N270X270

Commit message: Guitar Effects
Parts:
- added C12: 330p, Capacitor_SMD:C_0805_2012Metric, symbol Device:C
- C2: value 100n -> 10u
Connections:
- net MIC: now also C12.2
- net at R4.2, R5.1, U1.2 (-): now also C12.1
Changed lines of the file:
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@@
   (junction (at 48.895 81.28) (diameter 0) (color 0 0 0 0)
   )
+  (junction (at 250.19 85.09) (diameter 0) (color 0 0 0 0)
+  )
   (junction (at 232.41 71.755) (diameter 0) (color 0 0 0 0)
   )
@@
   (junction (at 144.78 77.47) (diameter 0) (color 0 0 0 0)
   )
+  (junction (at 264.16 85.09) (diameter 0) (color 0 0 0 0)
+  )
   (junction (at 266.7 74.295) (diameter 0) (color 0 0 0 0)
   )
@@
     (stroke (width 0) (type default))
   )
-  (wire (pts (xy 253.365 85.09) (xy 246.38 85.09))
+  (wire (pts (xy 253.365 85.09) (xy 250.19 85.09))
     (stroke (width 0) (type default))
   )
@@
     (stroke (width 0) (type default))
   )
+  (wire (pts (xy 264.16 95.25) (xy 264.16 85.09))
+    (stroke (width 0) (type default))
+  )
   (wire (pts (xy 93.98 54.61) (xy 93.98 57.15))
     (stroke (width 0) (type default))
   )
+  (wire (pts (xy 250.19 85.09) (xy 246.38 85.09))
+    (stroke (width 0) (type default))
+  )
   (wire (pts (xy 189.23 71.755) (xy 213.36 71.755))
     (stroke (width 0) (type default))
@@
     (stroke (width 0) (type default))
   )
+  (wire (pts (xy 260.985 95.25) (xy 264.16 95.25))
+    (stroke (width 0) (type default))
+  )
   (wire (pts (xy 60.325 57.15) (xy 64.135 57.15))
     (stroke (width 0) (type default))
@@
     (stroke (width 0) (type default))
   )
+  (wire (pts (xy 250.19 95.25) (xy 250.19 85.09))
+    (stroke (width 0) (type default))
+  )
   (wire (pts (xy 194.31 126.365) (xy 194.31 118.745))
     (stroke (width 0) (type default))
   )
-  (wire (pts (xy 260.985 85.09) (xy 266.7 85.09))
+  (wire (pts (xy 260.985 85.09) (xy 264.16 85.09))
     (stroke (width 0) (type default))
   )
@@
     (stroke (width 0) (type default))
   )
+  (wire (pts (xy 253.365 95.25) (xy 250.19 95.25))
+    (stroke (width 0) (type default))
+  )
   (wire (pts (xy 194.31 118.745) (xy 184.15 118.745))
     (stroke (width 0) (type default))
@@
   )
   (wire (pts (xy 58.42 119.38) (xy 58.42 124.46))
+    (stroke (width 0) (type default))
+  )
+  (wire (pts (xy 264.16 85.09) (xy 266.7 85.09))
     (stroke (width 0) (type default))
   )
@@
     )
   )
+  (symbol (lib_id "Device:C") (at 257.175 95.25 90) (unit 1)
+    (in_bom yes) (on_board yes) (dnp no)
+    (property "Reference" "C12" (at 257.175 88.8746 90)
+      (effects (font (size 1.27 1.27)))
+    )
+    (property "Value" "330p" (at 257.175 91.186 90)
+      (effects (font (size 1.27 1.27)))
+    )
+    (property "Footprint" "Capacitor_SMD:C_0805_2012Metric" (at 260.985 94.2848 0)
+      (effects (font (size 1.27 1.27)) hide)
+    )
+    (property "Datasheet" "~" (at 257.175 95.25 0)
+      (effects (font (size 1.27 1.27)) hide)
+    )
+    (pin "1")
+    (pin "2")
+    (instances
+      (project "things"
+        (path "/b6f73a49-ac1f-4895-a0f9-8f6954ee587f/52688484-ab73-49f2-b49e-ffc3daf8c274"
+          (reference "C12") (unit 1)
+        )
+      )
+      (project "audio"
+        (path "/de440898-6f94-46da-8c8e-7b125fe75199"
+          (reference "C?") (unit 1)
+        )
+      )
+    )
+  )
   (symbol (lib_id "power:GND") (at 93.98 86.36 0) (unit 1)
     (in_bom yes) (on_board yes) (dnp no)
@@
       (effects (font (size 1.27 1.27)) (justify left))
     )
-    (property "Value" "100n" (at 249.301 101.473 0)
-      (effects (font (size 1.27 1.27)) (justify left))
-    )
+    (property "Value" "10u" (at 249.301 101.473 0)
+      (effects (font (size 1.27 1.27)) (justify left))
+    )

Commit message: Add menu to guitar effects
Parts:
- added C13: 100n, Capacitor_SMD:C_0805_2012Metric, symbol Device:C
Connections:
- net GND: now also C13.1
- net at C3.2, R2.2, R3.1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: now also C13.2
Changed lines of the file:
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@@
   (junction (at 184.15 85.725) (diameter 0) (color 0 0 0 0)
   )
+  (junction (at 232.41 92.71) (diameter 0) (color 0 0 0 0)
+  )
   (junction (at 142.24 54.61) (diameter 0) (color 0 0 0 0)
   )
@@
   (junction (at 264.16 85.09) (diameter 0) (color 0 0 0 0)
   )
+  (junction (at 232.41 80.645) (diameter 0) (color 0 0 0 0)
+  )
   (junction (at 266.7 74.295) (diameter 0) (color 0 0 0 0)
   )
@@
     (stroke (width 0) (type default))
   )
+  (wire (pts (xy 232.41 80.645) (xy 232.41 83.185))
+    (stroke (width 0) (type default))
+  )
   (wire (pts (xy 109.22 62.23) (xy 82.55 62.23))
     (stroke (width 0) (type default))
@@
     (stroke (width 0) (type default))
   )
+  (wire (pts (xy 226.695 80.645) (xy 232.41 80.645))
+    (stroke (width 0) (type default))
+  )
   (wire (pts (xy 266.7 85.09) (xy 266.7 74.295))
     (stroke (width 0) (type default))
@@
     (stroke (width 0) (type default))
   )
-  (wire (pts (xy 232.41 90.805) (xy 232.41 93.98))
+  (wire (pts (xy 232.41 90.805) (xy 232.41 92.71))
     (stroke (width 0) (type default))
   )
@@
     (stroke (width 0) (type default))
   )
+  (wire (pts (xy 232.41 92.71) (xy 232.41 93.98))
+    (stroke (width 0) (type default))
+  )
   (wire (pts (xy 82.55 62.23) (xy 82.55 139.7))
     (stroke (width 0) (type default))
@@
     (stroke (width 0) (type default))
   )
+  (wire (pts (xy 226.695 83.185) (xy 226.695 80.645))
+    (stroke (width 0) (type default))
+  )
   (polyline (pts (xy 39.37 170.18) (xy 68.58 170.18))
     (stroke (width 0) (type default))
@@
     (stroke (width 0) (type default))
   )
+  (wire (pts (xy 226.695 90.805) (xy 226.695 92.71))
+    (stroke (width 0) (type default))
+  )
   (wire (pts (xy 253.365 95.25) (xy 250.19 95.25))
     (stroke (width 0) (type default))
@@
     (stroke (width 0) (type default))
   )
+  (wire (pts (xy 226.695 92.71) (xy 232.41 92.71))
+    (stroke (width 0) (type default))
+  )
   (wire (pts (xy 58.42 144.78) (xy 58.42 149.86))
     (stroke (width 0) (type default))
   )
-  (wire (pts (xy 232.41 76.835) (xy 232.41 83.185))
+  (wire (pts (xy 232.41 76.835) (xy 232.41 80.645))
     (stroke (width 0) (type default))
   )
@@
         )
       )
+    )
+  )
+  (symbol (lib_id "Device:C") (at 226.695 86.995 180) (unit 1)
+    (in_bom yes) (on_board yes) (dnp no)
+    (property "Reference" "C13" (at 220.3196 86.995 90)
+      (effects (font (size 1.27 1.27)))
+    )
+    (property "Value" "100n" (at 222.631 86.995 90)
+      (effects (font (size 1.27 1.27)))
+    )
+    (property "Footprint" "Capacitor_SMD:C_0805_2012Metric" (at 225.7298 83.185 0)
+      (effects (font (size 1.27 1.27)) hide)
+    )
+    (property "Datasheet" "~" (at 226.695 86.995 0)
+      (effects (font (size 1.27 1.27)) hide)
+    )
+    (pin "1")
+    (pin "2")
+    (instances
+      (project "things"
+        (path "/b6f73a49-ac1f-4895-a0f9-8f6954ee587f/52688484-ab73-49f2-b49e-ffc3daf8c274"
+          (reference "C13") (unit 1)
+        )
+      )
+      (project "audio"
+        (path "/de440898-6f94-46da-8c8e-7b125fe75199"
+          (reference "C?") (unit 1)
+        )
+      )

Commit message: Update docs for FM radio
Parts:
- added R? (x2): 1K, Resistor_SMD:R_0805_2012Metric, symbol Device:R
Connections:
- net GND: now also R?.2, R?.2
- net at J?.SN, U2.16 (INR+): now also R?.1
- net at J?.TN, U2.20 (INL+): now also R?.1
