File: 18_transmitter/schematic/transmitter.kicad_sch (KiCad schematic)
At the start: 14 parts, among them J3 max_9814 Module, J5 RF Out, U5 Pico

Commit message: Add amplifier experiments to transmitter
Parts:
- renumbered J5 to J1, J3 to J2, U5 to U7
Other:
- added sheet Amplifier (untitled.kicad_sch)
Changed lines of the file:
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@@
   (symbol (lib_id "pico:Pico") (at 215.9 90.17 0) (unit 1)
     (in_bom yes) (on_board yes) (dnp no) (fields_autoplaced)
-    (property "Reference" "U5" (at 215.9 58.42 0)
+    (property "Reference" "U7" (at 215.9 58.42 0)
       (effects (font (size 1.27 1.27)))
     )
@@
   (symbol (lib_id "Connector:Conn_01x05_Socket") (at 254 83.82 0) (unit 1)
     (in_bom yes) (on_board yes) (dnp no)
-    (property "Reference" "J3" (at 255.905 82.55 0)
+    (property "Reference" "J2" (at 255.905 82.55 0)
       (effects (font (size 1.27 1.27)) (justify left) hide)
     )
@@
   (symbol (lib_id "Connector:Conn_Coaxial") (at 25.4 86.36 0) (mirror y) (unit 1)
     (in_bom yes) (on_board yes) (dnp no)
-    (property "Reference" "J5" (at 21.59 85.3832 0)
+    (property "Reference" "J1" (at 21.59 85.3832 0)
       (effects (font (size 1.27 1.27)) (justify left) hide)
     )
@@
       )
     )
+  )
+  (sheet (at 30.48 21.59) (size 12.7 17.78) (fields_autoplaced)
+    (stroke (width 0.1524) (type solid))
+    (fill (color 0 0 0 0.0000))
+    (property "Sheetname" "Amplifier" (at 30.48 20.8784 0)
+      (effects (font (size 1.27 1.27)) (justify left bottom))
+    )
+    (property "Sheetfile" "untitled.kicad_sch" (at 30.48 39.9546 0)
+      (effects (font (size 1.27 1.27)) (justify left top))
+    )
+    (instances
+      (project "transmitter"
+        (path "/b6f73a49-ac1f-4895-a0f9-8f6954ee587f" (page "2"))
+      )
+    )

Commit message: tidy up transmit python script and transmitter.cpp example
Connections:
- net +3.3V: now reaches J2.4 (Pin_4), U7.36 (3V3)
Changed lines of the file:
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@@
   (junction (at 45.72 86.36) (diameter 0) (color 0 0 0 0)
+  )
+  (junction (at 245.745 76.2) (diameter 0) (color 0 0 0 0)
   )
   (junction (at 193.04 83.82) (diameter 0) (color 0 0 0 0)
@@
   )
   (wire (pts (xy 106.045 99.06) (xy 104.775 99.06))
+    (stroke (width 0) (type default))
+  )
+  (wire (pts (xy 245.745 66.04) (xy 245.745 76.2))
     (stroke (width 0) (type default))
   )
@@
         )
       )
+    )
+  )
+  (symbol (lib_id "power:+3.3V") (at 245.745 66.04 0) (unit 1)
+    (in_bom yes) (on_board yes) (dnp no) (fields_autoplaced)
+    (property "Reference" "#PWR03" (at 245.745 69.85 0)
+      (effects (font (size 1.27 1.27)) hide)
+    )
+    (property "Value" "+3.3V" (at 245.745 60.96 0)
+      (effects (font (size 1.27 1.27)))
+    )
+    (property "Footprint" "" (at 245.745 66.04 0)
+      (effects (font (size 1.27 1.27)) hide)
+    )
+    (property "Datasheet" "" (at 245.745 66.04 0)
+      (effects (font (size 1.27 1.27)) hide)
+    )
+    (pin "1")
+    (instances
+      (project "transmitter"
+        (path "/b6f73a49-ac1f-4895-a0f9-8f6954ee587f"
+          (reference "#PWR03") (unit 1)
+        )
+      )
