File: 19_fm_radio/schematic/fm_radio.kicad_sch (KiCad schematic)
At the start: 26 parts, among them J1 RDA7805 Module, J6 Antenna, J8 I2C Display, SW1 SW_SPDT, U2 TPA2012D2RTJT, U3 Pico

Commit message: Update docs for FM radio
Parts:
- added C? (x2): 10u, Capacitor_SMD:C_0805_2012Metric, symbol Device:C
- added C?: 100n, Capacitor_SMD:C_0805_2012Metric, symbol Device:C
- added FB?: Ferrite_Bead, Inductor_SMD:L_0805_2012Metric, symbol Device:Ferrite_Bead
- added R?: 10R, Resistor_SMD:R_0805_2012Metric, symbol Device:R
- renumbered J8 to J2, SW1 to SW6, U3 to U4
Connections:
- net +3V3: now also C?.2, FB?.2
- net +BATT: no longer J1.1 (Pin_1)
- net GND: now also C?.1, C?.1, C?.1
- new net: C?.2, C?.2, J1.1 (Pin_1), R?.1
- new net: FB?.1, R?.2
- no-connect marks 28 -> 27
Other:
- moved on the sheet: C?, J1, J6, J?, R?, U2
